File: cw308t_mspm0l2228/cw308t_mspm0l2228.kicad_sch (KiCad schematic)
At the start: 16 parts, among them J11 CW308_EAST_C, J7 CW308_WEST_A, J9 CW308_SOUTH_B, SW1 RESET, U1 MSPM0L2228SPN

Commit message: PCB: correct MSPM0L2228 package, no traces under the chip
- U1 footprint LQFP-80_14x14mm_P0.65mm -> LQFP-80_12x12mm_P0.5mm
  (TI PN0080A: 12x12 body, 14x14 over leads, 0.5mm pitch)
- Routing keepout under the chip body on both layers (VDD/GND crossed it)
- Re-routed: 0 unconnected, 0 clearance; 10 vias, none under U1
- Power 0.4mm, necked to 0.3mm at the 0.25mm QFP pads
- Regenerated CNC files, gerbers, renders; BOM/README/schematic updated

Co-Authored-By: Claude Opus 5.5 <noreply@anthropic.com>
Parts:
- U1: footprint Package_QFP:LQFP-80_14x14mm_P0.65mm -> Package_QFP:LQFP-80_12x12mm_P0.5mm
Changed lines of the file:
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@@
     (property "Reference" "U1" (at 200.5 146.86 0) (effects (font (size 1.27 1.27)) (justify left)))
     (property "Value" "MSPM0L2228SPN" (at 200.5 149.86 0) (effects (font (size 1.27 1.27)) (justify left)))
-    (property "Footprint" "Package_QFP:LQFP-80_14x14mm_P0.65mm" (at 190.5 149.86 0) (effects (font (size 1.27 1.27)) hide))
+    (property "Footprint" "Package_QFP:LQFP-80_12x12mm_P0.5mm" (at 190.5 149.86 0) (effects (font (size 1.27 1.27)) hide))
     (instances (project "cw308t_mspm0l2228" (path "/ROOT" (reference "U1") (unit 1)))))
   (symbol (lib_id "sca:CONN20") (at 90.17 139.7 0) (unit 1) (exclude_from_sim no) (in_bom yes) (on_board yes) (dnp no)
