File: pcb/pcb.kicad_sch (KiCad schematic)
At the start: 0 parts

Commit message: Added new pcb
Parts:
- added C1: 470nF, Capacitor_SMD:C_0805_2012Metric, symbol Device:C
- added C2: 10uF, Capacitor_SMD:C_0805_2012Metric, symbol Device:C
- added C3: 100nF, Capacitor_SMD:C_0805_2012Metric, symbol Device:C
- added C4: 4.7uF, Capacitor_SMD:C_0805_2012Metric, symbol Device:C
- added C5: 1uF, Capacitor_SMD:C_0805_2012Metric, symbol Device:C
- added C6: 10nF, Capacitor_SMD:C_0805_2012Metric, symbol Device:C
- added J1: CW308_WEST, Connector_PinSocket_2.54mm:PinSocket_1x20_P2.54mm_Vertical, symbol Connector_Generic:Conn_01x20
- added J3: CW308_EAST, Connector_PinSocket_2.54mm:PinSocket_1x20_P2.54mm_Vertical, symbol Connector_Generic:Conn_01x20
- added J4: CW308_SOUTH, Connector_PinSocket_2.54mm:PinSocket_1x20_P2.54mm_Vertical, symbol Connector_Generic:Conn_01x20
- added J5: DEBUG, Connector_PinHeader_2.54mm:PinHeader_1x08_P2.54mm_Vertical, symbol Connector:Conn_01x08_Pin
- added P1: WEST_PINS, Connector_PinHeader_2.54mm:PinHeader_1x20_P2.54mm_Vertical, symbol Connector_Generic:Conn_01x20
- added P3: EAST_PINS, Connector_PinHeader_2.54mm:PinHeader_1x20_P2.54mm_Vertical, symbol Connector_Generic:Conn_01x20
- added P4: SOUTH_PINS, Connector_PinHeader_2.54mm:PinHeader_1x20_P2.54mm_Vertical, symbol Connector_Generic:Conn_01x20
- added R1: 10R, Resistor_SMD:R_0805_2012Metric, symbol Device:R
- added R2, R4: 47k, Resistor_SMD:R_0805_2012Metric, symbol Device:R
- added R3: 4.7k, Resistor_SMD:R_0805_2012Metric, symbol Device:R
- added SW1: RESET, Button_Switch_SMD:SW_Push_1P1T_NO_CK_KMR2, symbol Switch:SW_Push
- added U1: MSPM0L2228SPMR, Package_QFP:LQFP-64_10x10mm_P0.5mm, symbol mspm0:MSPM0L2228SPMR
Connections:
- new net: J1.1 (Pin_1), P1.1 (Pin_1)
- new net: J1.10 (Pin_10), P1.10 (Pin_10), R3.2, U1.33 (PA0)
- new net: C6.1, J1.11 (Pin_11), J4.8 (Pin_8), J5.7 (Pin_7), P1.11 (Pin_11), P4.8 (Pin_8), R2.2, SW1.1, U1.38 (NRST)
- new net: J1.12 (Pin_12), P1.12 (Pin_12)
- new net: J1.13 (Pin_13), P1.13 (Pin_13)
- new net: J1.14 (Pin_14), P1.14 (Pin_14)
- new net: C1.2, C2.2, C3.2, C4.2, C5.2, C6.2, J1.15 (Pin_15), J1.16 (Pin_16), J1.2 (Pin_2), J1.4 (Pin_4), J1.6 (Pin_6), J3.1 (Pin_1), J3.10 (Pin_10), J3.16 (Pin_16), J3.17 (Pin_17), J3.4 (Pin_4), J3.7 (Pin_7), J3.9 (Pin_9), J4.1 (Pin_1), J4.10 (Pin_10), J4.9 (Pin_9), J5.2 (Pin_2), P1.15 (Pin_15), P1.16 (Pin_16), P1.2 (Pin_2), P1.4 (Pin_4), P1.6 (Pin_6), P3.1 (Pin_1), P3.10 (Pin_10), P3.16 (Pin_16), P3.17 (Pin_17), P3.4 (Pin_4), P3.7 (Pin_7), P3.9 (Pin_9), P4.1 (Pin_1), P4.10 (Pin_10), P4.9 (Pin_9), R4.2, SW1.2, U1.41 (VSS)
- new net: J1.17 (Pin_17), P1.17 (Pin_17)
- new net: J1.18 (Pin_18), P1.18 (Pin_18)
- new net: J1.19 (Pin_19), P1.19 (Pin_19)
- new net: J1.20 (Pin_20), J3.14 (Pin_14), J3.8 (Pin_8), J4.7 (Pin_7), P1.20 (Pin_20), P3.14 (Pin_14), P3.8 (Pin_8), P4.7 (Pin_7), R3.1
- new net: J1.3 (Pin_3), P1.3 (Pin_3), U1.46 (PA6)
- new net: J1.5 (Pin_5), P1.5 (Pin_5)
- new net: J1.7 (Pin_7), J5.5 (Pin_5), P1.7 (Pin_7), U1.56 (PA10/BSL_TX)
- new net: J1.8 (Pin_8), J5.6 (Pin_6), P1.8 (Pin_8), U1.57 (PA11/BSL_RX)
- new net: J1.9 (Pin_9), P1.9 (Pin_9)
- new net: J4.11 (Pin_11), P4.11 (Pin_11)
- new net: J4.12 (Pin_12), P4.12 (Pin_12)
- new net: J4.13 (Pin_13), P4.13 (Pin_13)
- new net: J4.14 (Pin_14), P4.14 (Pin_14)
- new net: J4.15 (Pin_15), P4.15 (Pin_15)
- new net: J4.16 (Pin_16), P4.16 (Pin_16)
- new net: J4.17 (Pin_17), P4.17 (Pin_17)
- new net: J4.18 (Pin_18), P4.18 (Pin_18)
- new net: J4.19 (Pin_19), P4.19 (Pin_19)
- new net: J4.2 (Pin_2), P4.2 (Pin_2)
- new net: J4.20 (Pin_20), P4.20 (Pin_20)
- new net: J4.3 (Pin_3), P4.3 (Pin_3)
- new net: J4.4 (Pin_4), P4.4 (Pin_4)
- new net: J4.5 (Pin_5), J5.3 (Pin_3), P4.5 (Pin_5), U1.12 (PA19/SWDIO)
- new net: J4.6 (Pin_6), J5.4 (Pin_4), P4.6 (Pin_6), U1.13 (PA20/SWCLK)
- new net: C4.1, J3.3 (Pin_3), J3.5 (Pin_5), J3.6 (Pin_6), P3.3 (Pin_3), P3.5 (Pin_5), P3.6 (Pin_6), R1.1
- new net: C2.1, C3.1, C5.1, J3.2 (Pin_2), J5.1 (Pin_1), P3.2 (Pin_2), R1.2, R2.1, U1.39 (VBAT), U1.40 (VDD)
- new net: C1.1, U1.32 (VCORE)
- new net: J3.11 (Pin_11), P3.11 (Pin_11)
- new net: J3.12 (Pin_12), P3.12 (Pin_12)
- new net: J3.13 (Pin_13), P3.13 (Pin_13)
- new net: J3.15 (Pin_15), P3.15 (Pin_15)
- new net: J3.18 (Pin_18), P3.18 (Pin_18)
- new net: J3.19 (Pin_19), P3.19 (Pin_19)
- new net: J3.20 (Pin_20), P3.20 (Pin_20)
- new net: J5.8 (Pin_8), R4.1, U1.11 (PA18/BSL_INVOKE)
- no-connect marks 0 -> 52
Other:
- title: (none) -> CW308 target - MSPM0L2228SPMR (LQFP-64)
