File: pcb/pcb.kicad_sch (KiCad schematic)
At the start: 19 parts, among them J1 CW308_WEST, J3 CW308_EAST, J4 CW308_SOUTH, J5 DEBUG, P1 WEST_PINS, P3 EAST_PINS, P4 SOUTH_PINS, SW1 RESET, U1 MSPM0L2228SPMR

Commit message: PCB: CNC-milled THT redesign, 1.0/0.5 mm, 8 wire jumpers, 3 mm fill isolation
Single-sided hat for the CW308-to-CW313 adapter, all copper on F.Cu, no vias.

- Through-hole parts: axial resistors, disc caps, 6 mm tactile switch.
- Milling rules (pcb.kicad_dru): 1.0 mm traces / 0.5 mm isolation; 0.3/0.2 mm only in the
  MSP fan-out area (MSP_FINE) and 0.35/0.2 mm between header pins (HDR_GAPS), 0.2 mm cutter.
  No-net copper fill keeps 3 mm from all copper, 1 mm minimum width, small islands removed.
- MSP pads lengthened to 0.3 x 2.5 mm for hand soldering.
- J5 reduced to 2 pins (BSL, GND); the debugger uses the P breakout headers.
- Trigger moved from PA0 to PB16 (MSP pin 4): firmware must follow.
- Outline widened to 62.5 x 72.05 mm (two traces fit outside the header rows).
- 8 wire jumpers with 12 dedicated holes; see pcb/wire-jumpers.md.
- CNC files (F.Cu, Edge.Cuts Gerbers with X2, Excellon drill) in pcb/cnc-files.

Co-Authored-By: Claude Opus 5.5 <noreply@anthropic.com>
Parts:
- C1, C2, C3, C4, C5, C6: footprint Capacitor_SMD:C_0805_2012Metric -> Capacitor_THT:C_Disc_D5.0mm_W2.5mm_P5.00mm
- J5: value DEBUG -> BSL_GND; footprint Connector_PinHeader_2.54mm:PinHeader_1x08_P2.54mm_Vertical -> Connector_PinHeader_2.54mm:PinHeader_1x02_P2.54mm_Vertical; symbol Connector:Conn_01x08_Pin -> Connector:Conn_01x02_Pin
- R1, R2, R3, R4: footprint Resistor_SMD:R_0805_2012Metric -> Resistor_THT:R_Axial_DIN0207_L6.3mm_D2.5mm_P7.62mm_Horizontal
- SW1: footprint Button_Switch_SMD:SW_Push_1P1T_NO_CK_KMR2 -> Button_Switch_THT:SW_PUSH_6mm
Connections:
- net TRIG: now reaches J1.10 (Pin_10), P1.10 (Pin_10), R3.2
- net TRIG: now also U1.4 (PB16); no longer U1.33 (PA0)
- net at C6.1, J1.11 (Pin_11), J4.8 (Pin_8)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: no longer J5.7 (Pin_7)
- net at J1.7 (Pin_7), P1.7 (Pin_7), U1.56 (PA10/BSL_TX): no longer J5.5 (Pin_5)
- net at J1.8 (Pin_8), P1.8 (Pin_8), U1.57 (PA11/BSL_RX): no longer J5.6 (Pin_6)
- net at J4.5 (Pin_5), P4.5 (Pin_5), U1.12 (PA19/SWDIO): no longer J5.3 (Pin_3)
- net at J4.6 (Pin_6), P4.6 (Pin_6), U1.13 (PA20/SWCLK): no longer J5.4 (Pin_4)
- net at C2.1, C3.1, C5.1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: no longer J5.1 (Pin_1)
- net at R4.1, U1.11 (PA18/BSL_INVOKE): now also J5.1 (Pin_1); no longer J5.8 (Pin_8)
